Commit message: PR06 intentional fault: attach lidar to camera with unchanged offset

File: src/course_description/urdf/vehicle.urdf.xacro (robot description, xacro)
@@ -61,5 +61,5 @@
   <xacro:sensor name="imu" size="0.03 0.03 0.02"/>
   <joint name="camera_joint" type="fixed"><parent link="base_link"/><child link="camera_link"/><origin xyz="0.28 0 0.38"/></joint>
-  <joint name="lidar_joint" type="fixed"><parent link="base_link"/><child link="lidar_link"/><origin xyz="0.28 0 0.38"/></joint>
+  <joint name="lidar_joint" type="fixed"><parent link="camera_link"/><child link="lidar_link"/><origin xyz="0.28 0 0.38"/></joint>
   <joint name="imu_joint" type="fixed"><parent link="base_link"/><child link="imu_link"/><origin xyz="0.28 0 0.38"/></joint>
 </robot>
